File: hardware/smd-star.sch (KiCad schematic (older format))
At the start: 15 parts, among them U1 NE555, U2 4017

Commit message: PCB Routed
Parts:
- added BT1: BK-883, BAT_BK-883, symbol smd-star:BK-883
- added D10, D9: LED, smd-star:LED_0805_2012Metric_Pad1.15x1.40mm_HandSolder, symbol smd-star:LED
- renumbered D8 to D1, D7 to D2, D6 to D3, D5 to D4, D4 to D5, D3 to D6, D2 to D7, D1 to D8
Connections:
- net LED0 is gone; now on net LED1: D1.2 (A), U2.3 (Q0)
- net +BATT: now also BT1.S1+, BT1.S2+
- net -BATT: now also U2.15 (Reset), BT1.-
- net LED1: no longer D2.2 (A), U2.2 (Q1)
- net LED2: now also D2.2 (A), U2.2 (Q1); no longer D3.2 (A), U2.4 (Q2)
- net LED3: now also D3.2 (A), U2.4 (Q2); no longer D4.2 (A), U2.7 (Q3)
- net LED4: now also D4.2 (A), U2.7 (Q3); no longer D5.2 (A), U2.10 (Q4)
- net LED5: now also D5.2 (A), U2.10 (Q4); no longer D6.2 (A), U2.1 (Q5)
- net LED6: now also D6.2 (A), U2.1 (Q5); no longer D7.2 (A), U2.5 (Q6)
- net LED7: now also D7.2 (A), U2.5 (Q6); no longer D8.2 (A), U2.6 (Q7)
- net LED_R: now also D10.1 (K), D9.1 (K)
- net LED10: now reaches U2.11 (Q9)
- net LED10: now also D10.2 (A)
- net RESET renamed LED9
- net LED9: now also D9.2 (A); no longer U2.15 (Reset)
- new net LED8: D8.2 (A), U2.6 (Q7)
- no-connect marks 2 -> 1
Other:
- moved on the sheet: D1, D2, D3, D4, D5, D6, D7, D8, R3
