File: hardware/smd-sun.kicad_pcb (KiCad board)
At the start: 2 copper layers, 50 x 50 mm, 19 parts, among them U1 NE555, U2 4017

Commit message: Rename all to smd-sun
Parts:
- BT1: footprint smd-star:BAT_BK-883 -> smd-sun:BAT_BK-883
- C1, C2: footprint smd-star:C_0805_2012Metric_Pad1.15x1.40mm_HandSolder -> smd-sun:C_0805_2012Metric_Pad1.15x1.40mm_HandSolder
- D1, D10, D2, D3, D4, D5, D6, D7, D8, D9: footprint smd-star:LED_0805_2012Metric_Pad1.15x1.40mm_HandSolder -> smd-sun:LED_0805_2012Metric_Pad1.15x1.40mm_HandSolder
- G***: footprint smd-star:mask_600 -> smd-sun:mask_600
- R1, R2, R3: footprint smd-star:R_0805_2012Metric_Pad1.15x1.40mm_HandSolder -> smd-sun:R_0805_2012Metric_Pad1.15x1.40mm_HandSolder
- U1: footprint smd-star:SO-8_3.9x4.9mm_P1.27mm -> smd-sun:SO-8_3.9x4.9mm_P1.27mm
- U2: footprint smd-star:SOIC-16_3.9x9.9mm_P1.27mm -> smd-sun:SOIC-16_3.9x9.9mm_P1.27mm
Changed lines of the file:
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@@
     (add_net "Net-(U1-Pad3)")
   )
-  (module smd-star:SOIC-16_3.9x9.9mm_P1.27mm (layer F.Cu)
+  (module smd-sun:SOIC-16_3.9x9.9mm_P1.27mm (layer F.Cu)
     (at 0 5 90)
     (descr "SOIC, 16 Pin (JEDEC MS-012AC, https://www.analog.com/media/en/package-pcb-resources/package/pkg_pdf/soic_narrow-r/r_16.pdf), generated with kicad-footprint-generator ipc_gullwing_generator.py")
@@
     )
   )
-  (module smd-star:SO-8_3.9x4.9mm_P1.27mm (layer F.Cu)
+  (module smd-sun:SO-8_3.9x4.9mm_P1.27mm (layer F.Cu)
     (at 0 -2.286)
     (descr "SO, 8 Pin (https://www.nxp.com/docs/en/data-sheet/PCF8523.pdf), generated with kicad-footprint-generator ipc_gullwing_generator.py")
@@
     )
   )
-  (module smd-star:BAT_BK-883 (layer B.Cu)
+  (module smd-sun:BAT_BK-883 (layer B.Cu)
     (at 0 1.016)
     (fp_text reference BT1 (at -7.69 10.605) (layer B.SilkS)
@@
     )
   )
-  (module smd-star:mask_600 (layer B.Cu)
+  (module smd-sun:mask_600 (layer B.Cu)
     (at 0.254 -8.89 180)
     (fp_text reference G*** (at 0 0) (layer B.SilkS) hide
@@
       (xy -0.313544 5.29543) (xy -0.01829 5.369762) (xy 0.322838 5.406304) (xy 0.679168 5.403443)) (layer B.SilkS) (width 0.01))
   )
-  (module smd-star:LED_0805_2012Metric_Pad1.15x1.40mm_HandSolder (layer F.Cu)
+  (module smd-sun:LED_0805_2012Metric_Pad1.15x1.40mm_HandSolder (layer F.Cu)
     (at 7 -7 170)
     (descr "LED SMD 0805 (2012 Metric), square (rectangular) end terminal, IPC_7351 nominal, (Body size source: https://docs.google.com/spreadsheets/d/1BsfQQcO9C6DZCsRaXUlFlo91Tg2WpOkGARC1WS5S8t0/edit?usp=sharing), generated with kicad-footprint-generator")
@@
     )
   )
-  (module smd-star:LED_0805_2012Metric_Pad1.15x1.40mm_HandSolder (layer F.Cu)
+  (module smd-sun:LED_0805_2012Metric_Pad1.15x1.40mm_HandSolder (layer F.Cu)
     (at -7 -7 10)
     (descr "LED SMD 0805 (2012 Metric), square (rectangular) end terminal, IPC_7351 nominal, (Body size source: https://docs.google.com/spreadsheets/d/1BsfQQcO9C6DZCsRaXUlFlo91Tg2WpOkGARC1WS5S8t0/edit?usp=sharing), generated with kicad-footprint-generator")
@@
     )
   )
-  (module smd-star:R_0805_2012Metric_Pad1.15x1.40mm_HandSolder (layer F.Cu)
+  (module smd-sun:R_0805_2012Metric_Pad1.15x1.40mm_HandSolder (layer F.Cu)
     (at 0 15.5)
     (descr "Resistor SMD 0805 (2012 Metric), square (rectangular) end terminal, IPC_7351 nominal with elongated pad for handsoldering. (Body size source: https://docs.google.com/spreadsheets/d/1BsfQQcO9C6DZCsRaXUlFlo91Tg2WpOkGARC1WS5S8t0/edit?usp=sharing), generated with kicad-footprint-generator")
@@
     )
   )
-  (module smd-star:R_0805_2012Metric_Pad1.15x1.40mm_HandSolder (layer F.Cu)
+  (module smd-sun:R_0805_2012Metric_Pad1.15x1.40mm_HandSolder (layer F.Cu)
     (at -6.6 4.064 90)
     (descr "Resistor SMD 0805 (2012 Metric), square (rectangular) end terminal, IPC_7351 nominal with elongated pad for handsoldering. (Body size source: https://docs.google.com/spreadsheets/d/1BsfQQcO9C6DZCsRaXUlFlo91Tg2WpOkGARC1WS5S8t0/edit?usp=sharing), generated with kicad-footprint-generator")
@@
     )
   )
-  (module smd-star:R_0805_2012Metric_Pad1.15x1.40mm_HandSolder (layer F.Cu)
+  (module smd-sun:R_0805_2012Metric_Pad1.15x1.40mm_HandSolder (layer F.Cu)
     (at 6.6 -0.254 270)
     (descr "Resistor SMD 0805 (2012 Metric), square (rectangular) end terminal, IPC_7351 nominal with elongated pad for handsoldering. (Body size source: https://docs.google.com/spreadsheets/d/1BsfQQcO9C6DZCsRaXUlFlo91Tg2WpOkGARC1WS5S8t0/edit?usp=sharing), generated with kicad-footprint-generator")
@@
     )
   )
-  (module smd-star:LED_0805_2012Metric_Pad1.15x1.40mm_HandSolder (layer F.Cu)
+  (module smd-sun:LED_0805_2012Metric_Pad1.15x1.40mm_HandSolder (layer F.Cu)
     (at 15.556 -15.556 225)
     (descr "LED SMD 0805 (2012 Metric), square (rectangular) end terminal, IPC_7351 nominal, (Body size source: https://docs.google.com/spreadsheets/d/1BsfQQcO9C6DZCsRaXUlFlo91Tg2WpOkGARC1WS5S8t0/edit?usp=sharing), generated with kicad-footprint-generator")
@@
     )
   )
-  (module smd-star:LED_0805_2012Metric_Pad1.15x1.40mm_HandSolder (layer F.Cu)
+  (module smd-sun:LED_0805_2012Metric_Pad1.15x1.40mm_HandSolder (layer F.Cu)
     (at 22 0 180)
     (descr "LED SMD 0805 (2012 Metric), square (rectangular) end terminal, IPC_7351 nominal, (Body size source: https://docs.google.com/spreadsheets/d/1BsfQQcO9C6DZCsRaXUlFlo91Tg2WpOkGARC1WS5S8t0/edit?usp=sharing), generated with kicad-footprint-generator")
@@
     )
   )
-  (module smd-star:LED_0805_2012Metric_Pad1.15x1.40mm_HandSolder (layer F.Cu)
+  (module smd-sun:LED_0805_2012Metric_Pad1.15x1.40mm_HandSolder (layer F.Cu)
     (at 15.556 15.556 135)
     (descr "LED SMD 0805 (2012 Metric), square (rectangular) end terminal, IPC_7351 nominal, (Body size source: https://docs.google.com/spreadsheets/d/1BsfQQcO9C6DZCsRaXUlFlo91Tg2WpOkGARC1WS5S8t0/edit?usp=sharing), generated with kicad-footprint-generator")
@@
     )
   )
-  (module smd-star:LED_0805_2012Metric_Pad1.15x1.40mm_HandSolder (layer F.Cu)
+  (module smd-sun:LED_0805_2012Metric_Pad1.15x1.40mm_HandSolder (layer F.Cu)
     (at 0 22 90)
     (descr "LED SMD 0805 (2012 Metric), square (rectangular) end terminal, IPC_7351 nominal, (Body size source: https://docs.google.com/spreadsheets/d/1BsfQQcO9C6DZCsRaXUlFlo91Tg2WpOkGARC1WS5S8t0/edit?usp=sharing), generated with kicad-footprint-generator")
@@
     )
   )
-  (module smd-star:LED_0805_2012Metric_Pad1.15x1.40mm_HandSolder (layer F.Cu)
+  (module smd-sun:LED_0805_2012Metric_Pad1.15x1.40mm_HandSolder (layer F.Cu)
     (at -15.556 15.556 45)
     (descr "LED SMD 0805 (2012 Metric), square (rectangular) end terminal, IPC_7351 nominal, (Body size source: https://docs.google.com/spreadsheets/d/1BsfQQcO9C6DZCsRaXUlFlo91Tg2WpOkGARC1WS5S8t0/edit?usp=sharing), generated with kicad-footprint-generator")
@@
     )
   )
-  (module smd-star:LED_0805_2012Metric_Pad1.15x1.40mm_HandSolder (layer F.Cu)
+  (module smd-sun:LED_0805_2012Metric_Pad1.15x1.40mm_HandSolder (layer F.Cu)
     (at -22 0)
     (descr "LED SMD 0805 (2012 Metric), square (rectangular) end terminal, IPC_7351 nominal, (Body size source: https://docs.google.com/spreadsheets/d/1BsfQQcO9C6DZCsRaXUlFlo91Tg2WpOkGARC1WS5S8t0/edit?usp=sharing), generated with kicad-footprint-generator")
@@
     )
   )
-  (module smd-star:LED_0805_2012Metric_Pad1.15x1.40mm_HandSolder (layer F.Cu)
+  (module smd-sun:LED_0805_2012Metric_Pad1.15x1.40mm_HandSolder (layer F.Cu)
     (at -15.556 -15.556 315)
     (descr "LED SMD 0805 (2012 Metric), square (rectangular) end terminal, IPC_7351 nominal, (Body size source: https://docs.google.com/spreadsheets/d/1BsfQQcO9C6DZCsRaXUlFlo91Tg2WpOkGARC1WS5S8t0/edit?usp=sharing), generated with kicad-footprint-generator")
@@
     )
   )
-  (module smd-star:LED_0805_2012Metric_Pad1.15x1.40mm_HandSolder (layer F.Cu)
+  (module smd-sun:LED_0805_2012Metric_Pad1.15x1.40mm_HandSolder (layer F.Cu)
     (at 0 -22 270)
     (descr "LED SMD 0805 (2012 Metric), square (rectangular) end terminal, IPC_7351 nominal, (Body size source: https://docs.google.com/spreadsheets/d/1BsfQQcO9C6DZCsRaXUlFlo91Tg2WpOkGARC1WS5S8t0/edit?usp=sharing), generated with kicad-footprint-generator")
@@
     )
   )
-  (module smd-star:C_0805_2012Metric_Pad1.15x1.40mm_HandSolder (layer F.Cu)
+  (module smd-sun:C_0805_2012Metric_Pad1.15x1.40mm_HandSolder (layer F.Cu)
     (at -6.6 -0.254 90)
     (descr "Capacitor SMD 0805 (2012 Metric), square (rectangular) end terminal, IPC_7351 nominal with elongated pad for handsoldering. (Body size source: https://docs.google.com/spreadsheets/d/1BsfQQcO9C6DZCsRaXUlFlo91Tg2WpOkGARC1WS5S8t0/edit?usp=sharing), generated with kicad-footprint-generator")
@@
     )
   )
-  (module smd-star:C_0805_2012Metric_Pad1.15x1.40mm_HandSolder (layer F.Cu)
+  (module smd-sun:C_0805_2012Metric_Pad1.15x1.40mm_HandSolder (layer F.Cu)
     (at 6.6 4.064 270)
     (descr "Capacitor SMD 0805 (2012 Metric), square (rectangular) end terminal, IPC_7351 nominal with elongated pad for handsoldering. (Body size source: https://docs.google.com/spreadsheets/d/1BsfQQcO9C6DZCsRaXUlFlo91Tg2WpOkGARC1WS5S8t0/edit?usp=sharing), generated with kicad-footprint-generator")
